File: pcb/helen-art.brd (EAGLE design)
At the start: 49.5 x 46 mm, 29 parts, among them IC1 TINY22S, IC2 MCP73811/2

Commit message: fix D+/D- swap and remove LED labels
Parts:
- moved R1 1.36 mm to (21.8, 8.89), turned to 180 degrees
- moved R2 0.83 mm to (24.8, 9.72)
Connections:
- removed net D+: IC1.2, R1.1
- removed net D-: IC1.3, R2.1
- new net N$3: IC1.3, R1.1
- new net N$4: IC1.2, R2.1
- net N$1: no longer R3.1
- net N$2: now also R3.1
Routing:
- net D-: track 32.9 -> 0.00 mm, vias 1 -> 0
- net N$3: track 0.00 -> 28.3 mm, vias 0 -> 1
- net N$4: track 0.00 -> 27.8 mm, vias 0 -> 1
- net D+: track 25.9 -> 0.00 mm, vias 1 -> 0
- net N$1: track 15.3 -> 5.17 mm, vias 2 -> 0
- net N$2: track 3.37 -> 7.26 mm
- net B2: track 87.9 -> 84.2 mm
- net BAT+: track 39.6 -> 41.1 mm
