File: pcb/helen-art.brd (EAGLE design)
At the start: 49.5 x 46 mm, 29 parts, among them IC1 TINY22S, IC2 MCP73811/2

Commit message: values for resistors
Parts:
- R1, R2: value (none) -> 68
- R3: value (none) -> 1.0k
